File: PCB/TetheredJoy.kicad_pcb (KiCad board)
At the start: 2 copper layers, 40 parts, among them J1 Conn_01x04, J10 Conn_01x02, J11 Conn_01x05, J12 Conn_01x04, J2 Conn_01x05, J3 Conn_01x02, J4 Conn_01x02, J5 Conn_01x02, J6 Conn_01x02, J7 Conn_01x02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

Commit message: PCB done
Parts:
- added H1: MountingHole_2.7mm_M2.5, MountingHole:MountingHole_2.7mm_M2.5, F.Cu at (201.9, 106.7)
- added H2: MountingHole_2.7mm_M2.5, MountingHole:MountingHole_2.7mm_M2.5, F.Cu at (221.0, 38.1)
- D4, D5, D6: footprint LED_SMD:LED_0805_2012Metric_Pad1.15x1.40mm_HandSolder -> LED_SMD:LED_1206_3216Metric_Pad1.42x1.75mm_HandSolder
- SW1, SW2, SW3, SW4: moved to B.Cu
- moved J1 77.3 mm to (215.3, 107.3), turned to 270 degrees
- moved J12 73.7 mm to (215.3, 103.5), turned to 270 degrees
- moved D7 63.2 mm to (219.1, 101.0), turned to 270 degrees
- moved C4 56.6 mm to (212.7, 94.6), turned to 180 degrees
- moved U1 51.2 mm to (213.4, 83.8)
- moved U2 50.0 mm to (216.5, 94.6)
- moved C3 47.8 mm to (215.3, 98.4), turned to 180 degrees
- moved D3 47.6 mm to (208.9, 65.4)
- moved SW4 42.3 mm to (208.9, 71.8)
- moved J10 41.5 mm to (221.0, 70.5)
- moved C1 41.0 mm to (200.7, 82.5), turned to 270 degrees
- moved D2 40.0 mm to (208.9, 57.8)
- moved J2 36.1 mm to (204.5, 78.7)
- moved R8 36.1 mm to (204.5, 50.2), turned to 90 degrees
- moved R7 33.2 mm to (201.9, 50.2), turned to 90 degrees
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Routing:
- net GND: track 0.00 -> 215.4 mm, vias 0 -> 3
- net +5V: track 0.00 -> 148.9 mm, vias 0 -> 6
- net LED1SW1: track 0.00 -> 65.9 mm, vias 0 -> 4
- net LED2SW2: track 0.00 -> 54.6 mm, vias 0 -> 5
- net Net-(J11-Pad3): track 0.00 -> 54.5 mm, vias 0 -> 2
- net Net-(D5-Pad2): track 0.00 -> 54.1 mm, vias 0 -> 2
- net LED3SW3: track 0.00 -> 49.6 mm, vias 0 -> 4
- net Net-(J11-Pad4): track 0.00 -> 48.0 mm, vias 0 -> 2
- net Net-(J11-Pad5): track 0.00 -> 46.6 mm, vias 0 -> 2
- net Net-(R8-Pad1): track 0.00 -> 45.6 mm, vias 0 -> 2
- net Net-(D4-Pad2): track 0.00 -> 44.6 mm, vias 0 -> 2
- net LED4SW4: track 0.00 -> 40.2 mm, vias 0 -> 4
- net Net-(R7-Pad1): track 0.00 -> 37.1 mm, vias 0 -> 2
- net TX: track 0.00 -> 28.3 mm, vias 0 -> 1
- net RX: track 0.00 -> 22.2 mm, vias 0 -> 1
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Other:
- board outline added: 26.7 x 76.2 mm
- board text added: "DMFE 2019"
- board text added: "T-Joy Rev nc"
